File: flight-controller/FlightController.kicad_sch (KiCad schematic)
At the start: 38 parts, among them J1 MSD-4-A, J2 Conn_01x03_Pin, J3 Conn_01x03_Pin, J4 Conn_01x03_Pin, J5 Conn_01x03_Pin, J6 USB4215-03-A_REVA, J7 Conn_01x03_Pin, J8 Conn_01x03_Pin, J9 Conn_01x04_Pin, U1 ESP32-S3-WROOM-1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

Commit message: switch usb port, add schottky diode
Parts:
- removed J6: USB4215-03-A_REVA, USB4215_03_A:GCT_USB4215-03-A_REVA, symbol USB4215-03-A_REVA:USB4215-03-A_REVA
- added C11: 100n, Capacitor_SMD:C_0603_1608Metric_Pad1.08x0.95mm_HandSolder, symbol Device:C
- added D2: SMAJ5.0A, Diode_SMD:D_SMA, symbol Diode:SMAJ5.0A
- added D3, D4: B5819W, Diode_SMD:D_SOD-123, symbol Device:D_Schottky
- added J10: GT-USB-7010B, GT-USB-7010B:G-SWITCH_GT-USB-7010B, symbol GT-USB-7010B:GT-USB-7010B
Connections:
- net +5V: now also D3.1 (K), D4.1 (K); no longer J2.2 (Pin_2)
- net 5V_USB: now also C11.2, D2.2 (A2), D3.2 (A), J10.A4_B9 (VBUS_A), J10.B4_A9 (VBUS_B)
- net DATA+: now also J10.A6 (D1+), J10.B6 (D2+)
- net DATA-: now also J10.A7 (D1-), J10.B7 (D2-)
- net GND: now also C11.1, D2.1 (A1), J10.A1_B12 (GND_A), J10.B1_A12 (GND_B), J10.SH1 (SHIELD), J10.SH2 (SHIELD), J10.SH3 (SHIELD), J10.SH4 (SHIELD)
- net CC2: now reaches CR1.1 (I/O1)
- net CC2: now also R3.2, J10.B5 (CC2)
- net CC1: now reaches CR1.3 (I/O2)
- net CC1: now also R4.2, J10.A5 (CC1)
- new net: D4.2 (A), J2.2 (Pin_2)
Other:
- moved on the sheet: R3, R4

Commit message: design files
Parts:
- added J6: Conn_01x04_Pin, Connector_PinHeader_2.54mm:PinHeader_1x04_P2.54mm_Vertical, symbol Connector:Conn_01x04_Pin
- R6, R7: value 2.7k -> 5.1k
Connections:
- net +3.3V: now also J6.4 (Pin_4)
- net GND: now also J6.3 (Pin_3)
- net I2C_SCL: now also J6.1 (Pin_1)
- net I2C_SDA: now also J6.2 (Pin_2)
